File: Controller/Fuel Cell Controller V1.sch (EAGLE design)
At the start: 65 parts, among them IC1 4081D, U1 ATMEGA328P_TQFP, U2 MAX3221CPWR, U3 ATMEGA328P_TQFP, U4 MAX3221CPWR

Commit message: update
Parts:
- removed C41, C42, C44: 0.33uF/12V, E-P-008-R1.2:C-USC0805
- removed C43: 0.047uF/12V, E-P-008-R1.2:C-USC0805
- removed U$4: DS3231, DS3231:DS3231
- removed U$9: LCD-BOARD, lcd board:LCD-BOARD
- added C13, C14, C15: 0.33uF/12V, E-P-008-R1.2:C-USC0805
- added C16: 0.047uF/12V, E-P-008-R1.2:C-USC0805
- added LCD1: LCD-BOARD, lcd board:LCD-BOARD
- added LED1, LED2, LED3, LED4, LED5, LED6, LED7, LED8: (no value), adafruit:LEDCHIPLED_0805
- added R10, R11, R12, R13, R15, R16, R17, R18, R19: 10k, SparkFun-Resistors:RESISTOR0805-RES
- added R14, R9: (no value), adafruit:R-US_R0603
- added R20, R21: 10k, adafruit:R-US_R0603
- added R22, R23, R24, R25, R26, R27, R28, R29: (no value), SparkFun-Resistors:RESISTOR0805-RES
- added R4: 4.7k, SparkFun-Resistors:RESISTOR0805-RES
- added R5, R6, R7, R8: 1M, SparkFun-Resistors:RESISTOR0805-RES
- added RTC1: DS3231, DS3231:DS3231
- added U5: MAX3221CPWR, Texas Instruments_By_element14_Batch_1:MAX3221CPWR
- added U6: SN74HC4040D, Texas Instruments_By_element14_Batch_1:SN74HC4040D
- C1, C3, C4: value (none) -> 0.33uF/12V; device adafruit:C-USC0603 -> E-P-008-R1.2:C-USC0805
- C10, C11, C12: value 0.33uF/12V -> (none); device E-P-008-R1.2:C-USC0805 -> adafruit:C-USC0603
- C6: value (none) -> 0.047uF/12V; device adafruit:C-USC0603 -> E-P-008-R1.2:C-USC0805
- C9: value 0.047uF/12V -> (none); device E-P-008-R1.2:C-USC0805 -> adafruit:C-USC0603
- R1: device adafruit:R-US_R0603 -> SparkFun-Resistors:RESISTOR0805-RES
- R2: value (none) -> 10k; device adafruit:R-US_R0603 -> SparkFun-Resistors:RESISTOR0805-RES
- R3: value (none) -> 4.7k; device adafruit:R-US_R0603 -> SparkFun-Resistors:RESISTOR0805-RES
- U1: value ATMEGA328P_TQFP -> SN74ALS153D; device SparkFun-DigitalIC:ATMEGA328P_TQFP -> Texas Instruments_By_element14_Batch_1:SN74ALS153D
- U4: value MAX3221CPWR -> ATMEGA328P_TQFP; device Texas Instruments_By_element14_Batch_1:MAX3221CPWR -> SparkFun-DigitalIC:ATMEGA328P_TQFP
- renumbered AUXPOWER to E1, CVM to ETH3, FCPOWER to E2, H2BOARD to ETH7, MOTOR_CTRL to ETH4, PRESSURE to ETH5, RELAY1 to ETH1, RELAY2 to ETH2, U$1 to T1, U$10 to S2, U$2 to O1, U$3 to SHT1, U$5 to CAN1, U$6 to S1, U$7 to FAN1, U$8 to M1, VALVES to ETH6
Connections:
- new net LED_CLK: T1.13/SCK/LED, U6.CLK
- new net MULTA: T1.3/CAN-TX/PWM, U1.A
- new net MULTB: T1.4/CAN-RX-PWM, U1.B
- new net MULTO1: R1.1, T1.5/PWM, U1.1Y
- new net MULTO2: R2.2, T1.2, U1.2Y
- new net M_SIG_1: ETH4.6, U1.2C2
- new net M_SIG_2: ETH4.7, U1.2C3
- new net N$28: R24.2, U6.QC
- new net N$29: R25.2, U6.QD
- new net N$30: R26.2, U6.QE
- new net N$31: R27.2, U6.QF
- new net N$32: R28.2, U6.QG
- new net N$33: R29.2, U6.QH
- new net N$34: U6.CLR, U6.QI
- new net N$35: LED5.A, R26.1
- new net N$36: LED6.A, R27.1
- new net N$37: LED7.A, R28.1
- new net N$38: LED8.A, R29.1
- net +3.3V: now also C10.1, C2.1, C5.1, C9.1, F1.2, LCD1.V, R14.2, R3.1, R4.1, R5.2, R6.2, R9.2, RTC1.3.3V, U4.AREF, U4.AVCC, U4.VCC@4, U4.VCC@6, U5.VCC, U6.VCC; no longer C3.1, C4.1, C7.1, C8.1, F9.2, R2.2, R3.2, U$4.3.3V, U$9.V, U1.AREF, U1.AVCC, U1.VCC@4, U1.VCC@6, U4.VCC
- net ATMEG1_RESET: now also R9.1, U3.PC6(/RESET); no longer R2.1, U1.PC6(/RESET)
- net ATMEG2_RESET: now also R14.1, U4.PC6(/RESET); no longer R3.1, U3.PC6(/RESET)
- net AUX12: now also F4.1, F9.1; no longer F1.1, F5.1
- net AUX5: now also F10.1; no longer F2.1
- net CAPCURR: now also R5.1
- net CAPVOLT: now also R7.1
- net CVMRX: now also U3.PD0(RXD); no longer U1.PD0(RXD)
- net CVMSIG1: now also R13.2, U1.1C0
- net CVMSIG2: now also R12.2, U1.1C1
- net CVMSIG3: now also R11.2, U1.1C2
- net CVMSIG4: now also R10.2, U1.1C3
- net CVMTX: now also U3.PD1(TXD); no longer U1.PD1(TXD)
- net CVM_SER_INVALID: now also U3.PD3(INT1); no longer U1.PD3(INT1)
- net EXTRA_SIG: now also R21.2, U1.2C1; no longer T1.5/PWM
- net EXTRA_V_G: now also R15.2
- net FC12: now also F5.1, F8.1; no longer F4.1, F7.1
- net FC5: now also F2.2, F6.1, F7.1, U1.VCC; no longer F10.1, F6.2, F8.1
- net FCCURR: now also R6.1
- net FCPRES: now also R19.1
- net FCVOLT: now also R8.1
- net GND: now also C10.2, C14.2, C15.2, C9.2, ETH5.SHD1, ETH5.SHD2, LCD1.GND, LED1.C, LED2.C, LED3.C, LED4.C, LED5.C, LED6.C, LED7.C, LED8.C, R1.2, R10.1, R11.1, R12.1, R13.1, R15.1, R16.1, R17.1, R18.1, R2.1, R20.1, R21.1, R7.2, R8.2, RTC1.GND, U1.1~G, U1.2~G, U1.GND, U4.AGND, U4.GND@3, U4.GND@5, U5.FORCEON, U5.GND, U5.~EN, U6.GND; no longer C1.2, C41.2, C42.2, C6.2, R1.1, U$4.GND, U$9.GND, U1.AGND, U1.GND@3, U1.GND@5, U4.FORCEON, U4.GND, U4.~EN
- net H2_OK: now also R20.2, U1.2C0; no longer R1.2, T1.2
- net MISO1: now also U3.PB4(MISO); no longer U1.PB4(MISO)
- net MISO2: now also U4.PB4(MISO); no longer U3.PB4(MISO)
- net MOSI1: now also U3.PB3(MOSI/OC2); no longer U1.PB3(MOSI/OC2)
- net MOSI2: now also U4.PB3(MOSI/OC2); no longer U3.PB3(MOSI/OC2)
- net MRX: now also U4.PD0(RXD), U5.ROUT; no longer U3.PD0(RXD), U4.ROUT
- net MRX12: now also U5.RIN; no longer U4.RIN
- net MTX: now also U4.PD1(TXD), U5.DIN; no longer U3.PD1(TXD), U4.DIN
- net MTX12: now also U5.DOUT; no longer U4.DOUT
- net M_SER_INVALID: now also U4.PD3(INT1), U5.~INVALID; no longer U3.PD3(INT1), U4.~INVALID
- net N$1: now also C11.1, U4.PB6(XTAL1/TOSC1); no longer C5.1, U3.PB6(XTAL1/TOSC1)
- net N$10: now also C15.1, U5.V-; no longer C12.1, U4.V-
- net N$11: now also F9.2; no longer F1.2
- net N$12: now also F10.2; no longer F2.2
- net N$13: now also F7.2; no longer F3.2
- net N$14: now also F8.2; no longer F4.2
- net N$15: now also F4.2; no longer F5.2
- net N$16: now also LED1.A, R22.1; no longer ETH5.4
- net N$17: now also R18.2, R19.2; no longer ETH5.5
- net N$18: now also LED2.A, R23.1; no longer ETH5.6
- net N$19: now also LED3.A, R24.1; no longer ETH5.7
- net N$2: now also C12.1, U4.PB7(XTAL2/TOSC2); no longer C6.1, U3.PB7(XTAL2/TOSC2)
- net N$20: now also LED4.A, R25.1; no longer ETH5.8
- net N$21: now also R22.2, U6.QA; no longer ETH5.SHD1
- net N$22: now also R23.2, U6.QB; no longer ETH5.SHD2
- net N$23: now also F2.1; no longer F6.1
- net N$24: now also F5.2; no longer F7.2
- net N$25: now also F6.2; no longer F8.2
- net N$26: now also F1.1; no longer F9.1
- net N$27: now also F3.2; no longer F10.2
- net N$3: now also C14.1, U5.V+; no longer C11.1, U4.V+
- net N$4: now also C7.1, U3.PB6(XTAL1/TOSC1); no longer C1.1, U1.PB6(XTAL1/TOSC1)
- net N$5: now also C8.1, U3.PB7(XTAL2/TOSC2); no longer C2.1, U1.PB7(XTAL2/TOSC2)
- net N$6: now also C16.1, U5.C1+; no longer C9.1, U4.C1+
- net N$7: now also C16.2, U5.C1-; no longer C9.2, U4.C1-
- net N$73: now also C3.1; no longer C41.1
- net N$74: now also C6.1; no longer C43.1
- net N$75: now also C6.2; no longer C43.2
- net N$76: now also C1.1; no longer C44.1
- net N$77: now also C1.2; no longer C44.2
- net N$78: now also C4.1; no longer C42.1
- net N$8: now also C13.1, U5.C2+; no longer C10.1, U4.C2+
- net N$9: now also C13.2, U5.C2-; no longer C10.2, U4.C2-
- net PURGE_V_G: now also R16.2
- net SCK1: now also U3.PB5(SCK); no longer U1.PB5(SCK)
- net SCK2: now also U4.PB5(SCK); no longer U3.PB5(SCK)
- net SCL: now also LCD1.SCL, R3.2, RTC1.SCL, U4.PC5(ADC5/SCL); no longer U$4.SCL, U$9.SCL, U1.PC5(ADC5/SCL)
- net SDA: now also LCD1.SDA, R4.2, RTC1.SDA, U4.PC4(ADC4/SDA); no longer U$4.SDA, U$9.SDA, U1.PC4(ADC4/SDA)
- net SUPPLY_V_G: now also R17.2
- net V+: now also U5.~FORCEOFF; no longer U4.~FORCEOFF
Other:
- note added: "It is faster"
- note added: "Output Is 5 Volts"
- note added: "Pressure Sensor Sensor"
- note added: "Use 74HC4040D instead"
- note removed: "to everything"

Commit message: main board routed
Parts:
- added C19: 0.1uF, adafruit:C-USC0603
- added C20: 10uF, adafruit:C-USC0603
- added FRAME7: FRAME-LETTERNO_PACKAGE, SparkFun-Aesthetics:FRAME-LETTERNO_PACKAGE
- added ISP3: AVRISP-BOX, adafruit:AVRISP-BOX
- added LED10, LED11, LED12, LED9: (no value), adafruit:LEDCHIPLED_0805
- added R30, R31, R32, R33, R34: 100, adafruit:R-US_R0603
- C10, C2: value (none) -> 10uF
- C11, C12, C7, C8: value (none) -> 22pF
- C5, C9: value (none) -> 0.1uF
- R14, R9: value (none) -> 10k
- R22: value (none) -> 10k; device SparkFun-Resistors:RESISTOR0805-RES -> adafruit:R-US_R0603
- R23, R24, R25, R26, R27, R28, R29: value (none) -> 100; device SparkFun-Resistors:RESISTOR0805-RES -> adafruit:R-US_R0603
- U6: value SN74HC4040D -> ATMEGA328P_TQFP; device Texas Instruments_By_element14_Batch_1:SN74HC4040D -> SparkFun-DigitalIC:ATMEGA328P_TQFP
Connections:
- removed net 5V: ETH2.5
- removed net AGND: T1.AGND
- removed net AREF: T1.AREF
- removed net GND1: ISP1.GND
- removed net LED_CLK: T1.13/SCK/LED, U6.CLK
- removed net N$17: R18.2, R19.2
- removed net V+: U2.~FORCEOFF, U5.~FORCEOFF
- new net ATMEG3_RESET: ISP3.RST, R22.1, U6.PC6(/RESET)
- new net MISO3: ISP3.MISO, U6.PB4(MISO)
- new net MOSI3: ISP3.MOSI, U6.PB3(MOSI/OC2)
- new net N$39: LED7.A, R29.1
- new net N$40: LED6.A, R28.1
- new net N$41: LED5.A, R27.1
- new net N$42: LED4.A, R26.1
- new net N$43: LED3.A, R25.1
- new net N$44: LED2.A, R24.1
- new net N$45: LED1.A, R23.1
- new net N$46: ETH5.3, R19.1
- new net SCK3: ISP3.SCK, U6.PB5(SCK)
- new net THIS_IS_NOT_CONNECTED_1: ISP1.VCC
- new net THIS_IS_NOT_CONNECTED_2: ISP2.VCC
- new net THIS_IS_NOT_CONNECTED_3: ISP3.VCC
- net +3.3V: now also C19.1, C20.1, R22.2, U2.~FORCEOFF, U5.~FORCEOFF, U6.AREF, U6.AVCC, U6.VCC@4, U6.VCC@6; no longer CAN1.VIN, U6.VCC
- net FC5: now also ETH2.5
- net FCPRES: now also R18.2, R19.2, T1.A11; no longer ETH5.3, R19.1, T1.23/A9/T/PWM
- net GND: now also C19.2, C20.2, ISP1.GND, ISP3.GND, LED10.C, LED11.C, LED12.C, LED9.C, U6.AGND, U6.GND@3, U6.GND@5; no longer U6.GND
- net N$16: now also R23.2, U6.PC0(ADC0); no longer LED1.A, R22.1
- net N$18: now also R24.2, U6.PC1(ADC1); no longer LED2.A, R23.1
- net N$19: now also R25.2, U6.PC2(ADC2); no longer LED3.A, R24.1
- net N$20: now also R26.2, U6.PC3(ADC3); no longer LED4.A, R25.1
- net N$21: now also R27.2, U6.ADC6; no longer R22.2, U6.QA
- net N$22: now also R28.2, U6.ADC7; no longer R23.2, U6.QB
- net N$28: now also R29.2, U6.PD0(RXD); no longer R24.2, U6.QC
- net N$29: now also R30.2, U6.PD1(TXD); no longer R25.2, U6.QD
- net N$30: now also R31.2, U6.PD2(INT0); no longer R26.2, U6.QE
- net N$31: now also R32.2, U6.PD3(INT1); no longer R27.2, U6.QF
- net N$32: now also R33.2, U6.PD4(XCK/T0); no longer R28.2, U6.QG
- net N$33: now also R34.2, U6.PD5(T1); no longer R29.2, U6.QH
- net N$34: now also LED12.A, R34.1; no longer U6.CLR, U6.QI
- net N$35: now also LED11.A, R33.1; no longer LED5.A, R26.1
- net N$36: now also LED10.A, R32.1; no longer LED6.A, R27.1
- net N$37: now also LED9.A, R31.1; no longer LED7.A, R28.1
- net N$38: now also R30.1; no longer R29.1
- net SCL: now also U6.PC5(ADC5/SCL)
- net SDA: now also U6.PC4(ADC4/SDA)
Other:
- note added: "Note: Check Atmega328p max current"
- note added: "STATUS LEDs"
- note removed: "It is faster"
- note removed: "Use 74HC4040D instead"
