File: Relay Board/Relay_Board.brd (EAGLE design)
At the start: 100 x 80 mm, 48 parts

Commit message: updated relay board
Parts:
- R12, R13, R14, R15: value (none) -> 10K
- moved U$16 3.43 mm to (7.78, 27.1)
- moved U$19 1.28 mm to (71.4, 65.3)
- moved U$10 0.84 mm to (53.5, 72.7)
Connections:
- net GND: no longer U$19.4
- net POWER_BOARD: no longer U$19.3
Routing:
- net GND: track 345.8 -> 399.5 mm, vias 6 -> 7
- net SUPERCAPS: track 23.0 -> 20.0 mm
- net 5V: track 139.1 -> 141.7 mm
- net POWER_BOARD: track 72.3 -> 70.0 mm
- net CAP_FUSE: track 98.7 -> 97.4 mm
- removed copper zone on layer 1, net CAP_FUSE
- removed copper zone on layer 16, net GND
