File: Relay Board/Relay_Board.sch (EAGLE design)
At the start: 46 parts

Commit message: update
Parts:
- removed U$16: MOSFET-SI6423DQ, MOSFET-S16423DQ:MOSFET-SI6423DQ
- added U$24: 732-3204-ND_CONNECTOR, Connector 732-3204:732-3204-ND_CONNECTOR
- added U$25: SI6926ADQ-T1-E3CT-ND_MOSFET, MOSFET Si6926ADQ:SI6926ADQ-T1-E3CT-ND_MOSFET
- U$1, U$10, U$13, U$14, U$2, U$20, U$23: value POWERCONNECTOR -> 732-3204-ND_CONNECTOR; device Connector-732-3200-ND:POWERCONNECTOR -> Connector 732-3204:732-3204-ND_CONNECTOR
- U$12: value MOSFET-SI6423DQ -> SHUNT_RESISTOR_CSM3637; device MOSFET-S16423DQ:MOSFET-SI6423DQ -> Vishay_Shunt_Resistor_CSM3637:SHUNT_RESISTOR_CSM3637
- U$19: value MOSFET-SI6423DQ -> 5555140-6; device MOSFET-S16423DQ:MOSFET-SI6423DQ -> 5555140-6 RJ11:5555140-6
- U$4: value FUSE_BLOCK_40A_500V_PCB_3555-2 -> SHUNT_RESISTOR_CSM3637; device FUSE_BLOCK_40A_500V_BLADE_PCB_3555-2:FUSE_BLOCK_40A_500V_PCB_3555-2 -> Vishay_Shunt_Resistor_CSM3637:SHUNT_RESISTOR_CSM3637
- U$9: value MOSFET-SI6423DQ -> SI6926ADQ-T1-E3CT-ND_MOSFET; device MOSFET-S16423DQ:MOSFET-SI6423DQ -> MOSFET Si6926ADQ:SI6926ADQ-T1-E3CT-ND_MOSFET
Connections:
- removed net N$2: U$5.CATHODE, U$6.A
- removed net N$27: U$21.D, U$4.1
- removed net N$4: U$10.1, U$4.2
- removed net N$6: R3.2, U$3.OUT
- removed net N$8: D3.C, U$15.85, U$16.SOURCE
- new net POWER_IN: U$1.P$1, U$4.A, U$6.A
- new net SHUNT_RES_1: U$4.D, U$5.ANODE, U$6.D
- new net SUPERCAPS: U$10.P$1, U$12.D, U$21.D
- net AUX12: no longer U$8.86
- net CAP_CURR: now also R3.2, U$3.OUT
- net CAP_FUSE: now also U$12.A
- net CAP_R: now also R13.2, U$9.G1; no longer R15.2, U$9.GATE
- net CHARGE_R: now also U$25.G2; no longer U$12.GATE
- net CHARGING_RES_NEG: now also U$14.P$1; no longer U$14.1
- net FC12: now also U$8.86
- net FC_CURR: now also R1.2, U$7.OUT
- net FC_POWER: now also U$13.P$1, U$5.CATHODE; no longer U$13.1, U$6.D
- net GND: now also U$19.4, U$19.5, U$19.6, U$19.SH1, U$19.SH2, U$2.P$1, U$23.P$1, U$24.P$1, U$25.S1, U$25.S2, U$9.S1, U$9.S2; no longer R1.1, R9.2, U$12.DRAIN, U$16.DRAIN, U$19.DRAIN, U$2.1, U$9.DRAIN
- net MOTOR: now also U$20.P$1; no longer U$20.1
- net MOTOR_R: now also U$9.G2; no longer U$19.GATE
- net N$1: now also R1.1, R9.2; no longer U$1.1, U$5.ANODE
- net N$29: now also U$9.D2; no longer U$19.SOURCE
- net N$3: now also D3.C, U$8.85, U$9.D1; no longer R1.2, U$7.OUT
- net N$5: now also U$15.85, U$25.D1; no longer U$8.85, U$9.SOURCE
- net N$7: now also U$25.D2; no longer U$12.SOURCE
- net POWER_BOARD: now also U$19.1, U$19.2, U$19.3; no longer U$23.1
- net START_R: now also R15.2, U$25.G1; no longer R13.2, U$16.GATE
- net V_IN_NEG_1: now also U$4.C
- net V_IN_NEG_2: now also U$12.C
- net V_IN_POS_1: now also U$4.B
- net V_IN_POS_2: now also U$12.B
Other:
- note added: "Cap GND"
- note added: "Motor GND"
- note removed: "PowerBoard"
- moved on the sheet: D1, D2, D3, D4, R12, R13, R14, R15

Commit message: updated relay board
Parts:
- R12, R13, R14, R15: value (none) -> 10K
Connections:
- net GND: no longer U$19.4
- net POWER_BOARD: no longer U$19.3
Changed lines of the file:
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@@
 <part name="U$21" library="Vishay_Shunt_Resistor_CSM3637" deviceset="SHUNT_RESISTOR_CSM3637" device=""/>
 <part name="U$22" library="Relay_CPC1907B" deviceset="RELAY-CPC1907B" device=""/>
-<part name="R12" library="SparkFun-Passives" deviceset="RESISTOR" device="0603-RES"/>
-<part name="R13" library="SparkFun-Passives" deviceset="RESISTOR" device="0603-RES"/>
-<part name="R14" library="SparkFun-Passives" deviceset="RESISTOR" device="0603-RES"/>
-<part name="R15" library="SparkFun-Passives" deviceset="RESISTOR" device="0603-RES"/>
+<part name="R12" library="SparkFun-Passives" deviceset="RESISTOR" device="0603-RES" value="10K"/>
+<part name="R13" library="SparkFun-Passives" deviceset="RESISTOR" device="0603-RES" value="10K"/>
+<part name="R14" library="SparkFun-Passives" deviceset="RESISTOR" device="0603-RES" value="10K"/>
+<part name="R15" library="SparkFun-Passives" deviceset="RESISTOR" device="0603-RES" value="10K"/>
 <part name="U$1" library="Connector 732-3204" deviceset="732-3204-ND_CONNECTOR" device=""/>
 <part name="U$2" library="Connector 732-3204" deviceset="732-3204-ND_CONNECTOR" device=""/>
@@
 <label x="177.8" y="213.36" size="1.778" layer="95" rot="R180"/>
 </segment>
-<segment>
-<pinref part="U$19" gate="G$1" pin="4"/>
-<wire x1="185.42" y1="231.14" x2="180.34" y2="231.14" width="0.1524" layer="91"/>
-<label x="172.72" y="231.14" size="1.778" layer="95"/>
-</segment>
 </net>
 <net name="FC_CURR" class="0">
@@
 <pinref part="ETH2" gate="G$1" pin="2"/>
 <wire x1="182.88" y1="117.475" x2="177.8" y2="117.475" width="0.1524" layer="91"/>
-<label x="167.64" y="117.475" size="1.778" layer="95"/>
+<label x="165.1" y="117.475" size="1.778" layer="95"/>
 </segment>
 <segment>
@@
 <label x="177.8" y="243.84" size="1.778" layer="95" rot="R180"/>
 </segment>
-<segment>
-<pinref part="U$19" gate="G$1" pin="3"/>
-<wire x1="185.42" y1="236.22" x2="180.34" y2="236.22" width="0.1524" layer="91"/>
-<label x="160.02" y="236.22" size="1.778" layer="95"/>
-</segment>
 </net>
 <net name="N$1" class="0">
@@
 <pinref part="ETH2" gate="G$1" pin="1"/>
 <wire x1="182.88" y1="120.015" x2="177.8" y2="120.015" width="0.1524" layer="91"/>
-<label x="165.735" y="120.015" size="1.778" layer="95"/>
-</segment>
-<segment>
+<label x="163.195" y="120.015" size="1.778" layer="95"/>
+</segment>
+<segment>
