File: CVM Board/Archive/ecocar_CVM.brd (EAGLE design)
At the start: 110.2 x 92.7 mm, 148 parts, among them U2 MAX3221CPWR

Commit message: couple board revisions
Other:
- board text added: "UABERTA ECOCAR Cell VM BOARD"
- board text removed: "UABERTA ECOCAR CVM BOARD"
Changed lines of the file:
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@@
 <text x="89.535" y="21.59" size="0.7" layer="21" font="vector" ratio="15">V46</text>
 <text x="90.805" y="15.875" size="0.7" layer="21" font="vector" ratio="15">GND</text>
-<text x="47.117" y="89.027" size="1.27" layer="21" font="vector" ratio="15">UABERTA ECOCAR CVM BOARD</text>
+<text x="47.117" y="89.027" size="1.27" layer="21" font="vector" ratio="15">UABERTA ECOCAR Cell VM BOARD</text>
 </plain>
 <attributes>
