File: Hardware/FCC Power Board/fc power board.brd (EAGLE design)
At the start: 100 x 50 mm, 32 parts

Commit message: update
Parts:
- added STANDOFF1, STANDOFF2, STANDOFF3, STANDOFF4: STAND-OFF, SparkFun-Electromechanical:STAND-OFF
- moved U$8 69.2 mm to (81.3, -2.54), turned to 180 degrees
- moved U$9 55.2 mm to (95.2, 15.2), turned to 270 degrees
- moved R1 40.2 mm to (61.0, 20.3), flipped to the bottom, turned to 270 degrees
- moved L2 37.5 mm to (90.2, 17.8)
- moved R19 36.1 mm to (55.9, 20.3), flipped to the bottom, turned to 270 degrees
- moved LED1 34.0 mm to (61.0, 29.2), turned to 90 degrees
- moved R18 33.7 mm to (50.8, 20.3), flipped to the bottom, turned to 90 degrees
- moved C4 30.5 mm to (78.7, 17.8), turned to 180 degrees
- moved LED6 29.0 mm to (55.9, 29.2), turned to 90 degrees
- moved C7 28.1 mm to (75.9, 30.5), turned to 90 degrees
- moved R17 28.0 mm to (45.7, 20.3), flipped to the bottom, turned to 270 degrees
- moved R2 27.4 mm to (40.6, 20.3), flipped to the bottom, turned to 270 degrees
- moved LED5 25.2 mm to (50.8, 29.2), turned to 90 degrees
- moved D2 23.9 mm to (95.2, 27.9), turned to 270 degrees
- moved U$3 22.8 mm to (21.6, 27.9), turned to 180 degrees
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Connections:
- removed net FC_GND: U$5.P$2, U$5.P$3
- net GND: now also U$5.P$2, U$5.P$3
Routing:
- net FC_GND: track 54.7 -> 0.00 mm
- net GND: track 8.07 -> 50.0 mm, vias 1 -> 4
- net 5V_OUT: track 0.00 -> 33.8 mm
- net 12V_OUT: track 60.8 -> 82.0 mm, vias 1 -> 2
- net FC_IN: track 0.00 -> 19.1 mm
- net N$16: track 0.00 -> 16.7 mm
- net BATT_12V: track 42.8 -> 59.2 mm
- net 5V: track 0.00 -> 14.3 mm
- net FC_48V: track 27.2 -> 19.4 mm
- net N$17: track 0.00 -> 6.44 mm, vias 0 -> 1
- net N$4: track 2.75 -> 6.44 mm, vias 0 -> 1
- net N$3: track 2.75 -> 6.44 mm, vias 0 -> 1
- net N$24: track 2.75 -> 6.44 mm, vias 0 -> 1
- net N$21: track 2.75 -> 6.44 mm, vias 0 -> 1
- net 12V: track 0.00 -> 2.54 mm
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- added copper zone on layer 16, net 5V_OUT
- removed copper zone on layer 1, net BATT_12V
- removed copper zone on layer 1, net FC_12V
- removed copper zone on layer 1, net FC_GND
- removed copper zone on layer 1, net FC_IN
Other:
- board size 100 x 50 mm -> 100 x 49.5 mm
- board text added: "12V"
- board text added: "12v"
- board text added: "12v-b"
- board text added: "12v-fc"
- board text added: "48v-fc"
- board text added: "5V"
- board text added: "5v"
- board text removed: "+12V"
- board text removed: "+5V"
- board text removed: "12V_OUT"
- board text removed: "5V_OUT"
- board text removed: "BATT"
- board text removed: "BATT_12V"
- board text removed: "E-P-204-R3.4 Power Board University of Alberta EcoCar Team"
- board text removed: "FC+"
- board text removed: "FC-"
- board text removed: "FC_12V"
- board text removed: "FC_48V"
