File: Hardware/FCC Power Board/fc power board.sch (EAGLE design)
At the start: 32 parts

Commit message: update
Parts:
- added STANDOFF1, STANDOFF2, STANDOFF3, STANDOFF4: STAND-OFF, SparkFun-Electromechanical:STAND-OFF
Connections:
- removed net FC_GND: U$5.-VIN, U$5.ON/OFF
- net GND: now also U$5.-VIN, U$5.ON/OFF
Other:
- moved on the sheet: C4, C7, L2, LED5, R18
Changed lines of the file:
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@@
 <?xml version="1.0" encoding="utf-8"?>
 <!DOCTYPE eagle SYSTEM "eagle.dtd">
-<eagle version="7.7.0">
+<eagle version="7.4.0">
 <drawing>
 <settings>
@@
 <setting verticaltext="up"/>
 </settings>
-<grid distance="0.05" unitdist="inch" unit="inch" style="lines" multiple="1" display="no" altdistance="0.01" altunitdist="inch" altunit="inch"/>
+<grid distance="0.1" unitdist="inch" unit="inch" style="lines" multiple="1" display="no" altdistance="0.01" altunitdist="inch" altunit="inch"/>
 <layers>
 <layer number="1" name="Top" color="4" fill="1" visible="no" active="no"/>
@@
 <part name="U$9" library="MURS120T3G" deviceset="MURS120T3G" device=""/>
 <part name="PE11" library="supply1" deviceset="GND" device=""/>
+<part name="FRAME1" library="frames" deviceset="A3L-LOC" device=""/>
+<part name="STANDOFF1" library="SparkFun-Electromechanical" deviceset="STAND-OFF" device=""/>
+<part name="STANDOFF2" library="SparkFun-Electromechanical" deviceset="STAND-OFF" device=""/>
+<part name="STANDOFF3" library="SparkFun-Electromechanical" deviceset="STAND-OFF" device=""/>
+<part name="STANDOFF4" library="SparkFun-Electromechanical" deviceset="STAND-OFF" device=""/>
+<part name="GND3" library="supply1" deviceset="GND" device=""/>
 </parts>
 <sheets>
@@
 <text x="91.44" y="33.02" size="1.778" layer="91">Fuel Cell 12V Output\</text>
 <text x="104.14" y="-48.26" size="1.778" layer="91">12V Output</text>
-<text x="107.95" y="55.88" size="1.778" layer="91">5 Volt Connected</text>
+<text x="-128.27" y="-58.42" size="1.778" layer="91">5 Volt Connected</text>
 </plain>
 <instances>
@@
 <instance part="PE15" gate="1" x="83.82" y="25.4"/>
 <instance part="R17" gate="G$1" x="83.82" y="45.72" rot="R90"/>
-<instance part="LED5" gate="G$1" x="130.81" y="55.88" rot="R180"/>
-<instance part="PE16" gate="1" x="130.81" y="64.77" rot="R180"/>
-<instance part="R18" gate="G$1" x="130.81" y="45.72" rot="R90"/>
+<instance part="LED5" gate="G$1" x="-100.33" y="-58.42" rot="R180"/>
+<instance part="PE16" gate="1" x="-100.33" y="-49.53" rot="R180"/>
+<instance part="R18" gate="G$1" x="-100.33" y="-68.58" rot="R90"/>
 <instance part="LED6" gate="G$1" x="99.06" y="-45.72"/>
 <instance part="PE17" gate="1" x="99.06" y="-58.42"/>
@@
 <instance part="U$11" gate="G$1" x="-132.08" y="40.64" rot="R180"/>
 <instance part="U$6" gate="G$1" x="-132.08" y="-5.08" rot="R180"/>
-<instance part="U$8" gate="A" x="163.83" y="38.1"/>
-<instance part="L2" gate="G$1" x="146.05" y="38.1" rot="R90"/>
-<instance part="C4" gate="G$1" x="130.81" y="33.02"/>
-<instance part="C7" gate="G$1" x="156.21" y="30.48"/>
-<instance part="PE7" gate="1" x="130.81" y="25.4"/>
-<instance part="PE8" gate="1" x="156.21" y="22.86"/>
-<instance part="PE9" gate="1" x="245.11" y="30.48"/>
-<instance part="PE10" gate="1" x="262.89" y="35.56"/>
-<instance part="U$9" gate="G$1" x="158.75" y="43.18" rot="R270"/>
-<instance part="PE11" gate="1" x="158.75" y="55.88" rot="R180"/>
+<instance part="U$8" gate="A" x="-67.31" y="-76.2"/>
+<instance part="L2" gate="G$1" x="-85.09" y="-76.2" rot="R90"/>
+<instance part="C4" gate="G$1" x="-100.33" y="-81.28"/>
+<instance part="C7" gate="G$1" x="-74.93" y="-83.82"/>
+<instance part="PE7" gate="1" x="-100.33" y="-88.9"/>
+<instance part="PE8" gate="1" x="-74.93" y="-91.44"/>
+<instance part="PE9" gate="1" x="13.97" y="-83.82"/>
+<instance part="PE10" gate="1" x="31.75" y="-78.74"/>
+<instance part="U$9" gate="G$1" x="-72.39" y="-71.12" rot="R270"/>
+<instance part="PE11" gate="1" x="-72.39" y="-58.42" rot="R180"/>
+<instance part="FRAME1" gate="G$1" x="-193.04" y="-121.92"/>
+<instance part="STANDOFF1" gate="G$1" x="-167.64" y="-17.78"/>
+<instance part="STANDOFF2" gate="G$1" x="-167.64" y="-22.86"/>
+<instance part="STANDOFF3" gate="G$1" x="-167.64" y="-27.94"/>
+<instance part="STANDOFF4" gate="G$1" x="-167.64" y="-33.02"/>
+<instance part="GND3" gate="1" x="17.78" y="43.18" rot="R270"/>
 </instances>
 <busses>
@@
 <segment>
 <pinref part="U$8" gate="A" pin="VIN"/>
-<wire x1="163.83" y1="35.56" x2="156.21" y2="35.56" width="0.1524" layer="91"/>
+<wire x1="-67.31" y1="-78.74" x2="-74.93" y2="-78.74" width="0.1524" layer="91"/>
 <pinref part="C7" gate="G$1" pin="1"/>
-<wire x1="156.21" y1="35.56" x2="146.05" y2="35.56" width="0.1524" layer="91"/>
-<junction x="156.21" y="35.56"/>
-<label x="143.51" y="33.02" size="1.778" layer="95"/>
+<wire x1="-74.93" y1="-78.74" x2="-85.09" y2="-78.74" width="0.1524" layer="91"/>
+<junction x="-74.93" y="-78.74"/>
+<label x="-87.63" y="-81.28" size="1.778" layer="95"/>
 </segment>
 </net>
@@
 <pinref part="U$8" gate="A" pin="~ON~/OFF"/>
 <pinref part="PE10" gate="1" pin="GND"/>
-<wire x1="234.95" y1="38.1" x2="262.89" y2="38.1" width="0.1524" layer="91"/>
+<wire x1="3.81" y1="-76.2" x2="31.75" y2="-76.2" width="0.1524" layer="91"/>
 </segment>
 <segment>
 <pinref part="U$8" gate="A" pin="GND"/>
-<wire x1="234.95" y1="33.02" x2="245.11" y2="33.02" width="0.1524" layer="91"/>
+<wire x1="3.81" y1="-81.28" x2="13.97" y2="-81.28" width="0.1524" layer="91"/>
 <pinref part="PE9" gate="1" pin="GND"/>
 </segment>
 <segment>
 <pinref part="C4" gate="G$1" pin="2"/>
-<wire x1="130.81" y1="30.48" x2="130.81" y2="27.94" width="0.1524" layer="91"/>
+<wire x1="-100.33" y1="-83.82" x2="-100.33" y2="-86.36" width="0.1524" layer="91"/>
 <pinref part="PE7" gate="1" pin="GND"/>
 </segment>
 <segment>
 <pinref part="C7" gate="G$1" pin="2"/>
-<wire x1="156.21" y1="27.94" x2="156.21" y2="25.4" width="0.1524" layer="91"/>
+<wire x1="-74.93" y1="-86.36" x2="-74.93" y2="-88.9" width="0.1524" layer="91"/>
 <pinref part="PE8" gate="1" pin="GND"/>
 </segment>
 <segment>
 <pinref part="U$9" gate="G$1" pin="PIN1"/>
-<wire x1="158.75" y1="50.8" x2="158.75" y2="53.34" width="0.1524" layer="91"/>
+<wire x1="-72.39" y1="-63.5" x2="-72.39" y2="-60.96" width="0.1524" layer="91"/>
 <pinref part="PE11" gate="1" pin="GND"/>
 </segment>
@@
 <pinref part="PE16" gate="1" pin="GND"/>
 <pinref part="LED5" gate="G$1" pin="C"/>
-<wire x1="130.81" y1="62.23" x2="130.81" y2="60.96" width="0.1524" layer="91"/>
+<wire x1="-100.33" y1="-52.07" x2="-100.33" y2="-53.34" width="0.1524" layer="91"/>
+</segment>
+<segment>
+<pinref part="U$5" gate="G$1" pin="-VIN"/>
+<wire x1="35.56" y1="43.18" x2="20.32" y2="43.18" width="0.1524" layer="91"/>
+<label x="20.32" y="43.18" size="1.778" layer="95"/>
+<pinref part="U$5" gate="G$1" pin="ON/OFF"/>
+<wire x1="35.56" y1="48.26" x2="35.56" y2="43.18" width="0.1524" layer="91"/>
+<junction x="35.56" y="43.18"/>
+<pinref part="GND3" gate="1" pin="GND"/>
 </segment>
 </net>
@@
 <pinref part="C4" gate="G$1" pin="1"/>
 <pinref part="L2" gate="G$1" pin="1"/>
-<wire x1="130.81" y1="38.1" x2="138.43" y2="38.1" width="0.1524" layer="91"/>
-<wire x1="130.81" y1="38.1" x2="123.19" y2="38.1" width="0.1524" layer="91"/>
-<junction x="130.81" y="38.1"/>
-<label x="123.19" y="38.1" size="1.778" layer="95"/>
+<wire x1="-100.33" y1="-76.2" x2="-92.71" y2="-76.2" width="0.1524" layer="91"/>
+<wire x1="-100.33" y1="-76.2" x2="-107.95" y2="-76.2" width="0.1524" layer="91"/>
+<junction x="-100.33" y="-76.2"/>
+<label x="-107.95" y="-76.2" size="1.778" layer="95"/>
 <pinref part="R18" gate="G$1" pin="1"/>
-<wire x1="130.81" y1="40.64" x2="130.81" y2="38.1" width="0.1524" layer="91"/>
+<wire x1="-100.33" y1="-73.66" x2="-100.33" y2="-76.2" width="0.1524" layer="91"/>
 </segment>
 <segment>
 <pinref part="U$8" gate="A" pin="FB"/>
-<wire x1="234.95" y1="35.56" x2="245.11" y2="35.56" width="0.1524" layer="91"/>
-<label x="245.11" y="35.56" size="1.778" layer="95"/>
+<wire x1="3.81" y1="-78.74" x2="13.97" y2="-78.74" width="0.1524" layer="91"/>
+<label x="13.97" y="-78.74" size="1.778" layer="95"/>
 </segment>
 </net>
@@
 </segment>
 </net>
-<net name="FC_GND" class="0">
-<segment>
-<pinref part="U$5" gate="G$1" pin="-VIN"/>
-<wire x1="35.56" y1="43.18" x2="20.32" y2="43.18" width="0.1524" layer="91"/>
-<label x="20.32" y="43.18" size="1.778" layer="95"/>
-<pinref part="U$5" gate="G$1" pin="ON/OFF"/>
-<wire x1="35.56" y1="48.26" x2="35.56" y2="43.18" width="0.1524" layer="91"/>
-<junction x="35.56" y="43.18"/>
-</segment>
-</net>
 <net name="FC_IN" class="0">
 <segment>
@@
 <segment>
 <pinref part="U$8" gate="A" pin="OUTOUT"/>
-<wire x1="163.83" y1="38.1" x2="158.75" y2="38.1" width="0.1524" layer="91"/>
+<wire x1="-67.31" y1="-76.2" x2="-72.39" y2="-76.2" width="0.1524" layer="91"/>
 <pinref part="L2" gate="G$1" pin="2"/>
 <pinref part="U$9" gate="G$1" pin="P$2"/>
-<wire x1="158.75" y1="38.1" x2="153.67" y2="38.1" width="0.1524" layer="91"/>
-<junction x="158.75" y="38.1"/>
+<wire x1="-72.39" y1="-76.2" x2="-77.47" y2="-76.2" width="0.1524" layer="91"/>
+<junction x="-72.39" y="-76.2"/>
 </segment>
 </net>
@@
 <pinref part="LED5" gate="G$1" pin="A"/>
 <pinref part="R18" gate="G$1" pin="2"/>
-<wire x1="130.81" y1="53.34" x2="130.81" y2="50.8" width="0.1524" layer="91"/>
-</segment>
-</net>
+<wire x1="-100.33" y1="-60.96" x2="-100.33" y2="-63.5" width="0.1524" layer="91"/>
+</segment>
+</net>
