File: Hardware/Mosfet Board/mosfet board_v2.sch (EAGLE design)
At the start: 26 parts, among them IC1 4081D, U1 MOSFET1, U2 MOSFET2, U3 MOSFET3

Commit message: new independent mosfet board
Parts:
- removed C1: (no value), E-P-008-R1.2:C-USC0603
- removed D1: D1, diode:1N4004
- removed D2: D2, diode:1N4004
- removed D3: D3, diode:1N4004
- removed F1, F2, F3: (no value), polyfuse:POLYFUSE
- removed IC1: 4081D, 40xx:4081D
- removed JP1, JP2: (no value), adafruit:PINHD-1X6
- removed LED1, LED2, LED3: (no value), adafruit:LEDCHIPLED_0603
- removed U1: MOSFET1, MOSFET:MOSFET
- removed U2: MOSFET2, MOSFET:MOSFET
- removed U3: MOSFET3, MOSFET:MOSFET
- added E1: AUX PWR, 5555140-6 RJ11:5555140-6
- added E2: FC PWR, 5555140-6 RJ11:5555140-6
- added ETH1, ETH2, ETH3: ETHERNET, ETHERNET:ETHERNET
- added FRAME1, FRAME2: FRAME-LETTERNO_PACKAGE, FRAME-LETTER:FRAME-LETTERNO_PACKAGE
- added J1, J2, J3: (no value), SparkFun-Connectors:PINHD-2X3
- added Q1, Q2, Q3, Q4, Q5, Q6, Q7: MOSFET-NCH-AO3404A, n-mos switch:MOSFET-NCH-AO3404A
- added R11, R13, R18, R20: 10k, Resistor:RESISTOR0805
- added R12, R14, R19, R21: 100, Resistor:RESISTOR0805
- added R15, R16, R17, R22, R23: 1k, Resistor:RESISTOR0805
- added U$1, U$2, U$3, U$4, U$5, U$6, U$7: 656, GlassFuseHolder:656
- added U$10, U$12, U$14, U$16, U$18, U$20, U$8: H11L1M, H11L1M:H11L1M
- added U$11, U$13, U$15, U$17, U$19, U$21, U$9: SN74LVC1G04-Q1, SN74LVC1G04-Q1:SN74LVC1G04-Q1
- R1: value R1 -> 100; device resistor:R-US_R0603 -> Resistor:RESISTOR0805
- R10: value 10k -> 1k; device adafruit:R-US_R0603 -> Resistor:RESISTOR0805
- R2: value R2 -> 10k; device resistor:R-US_R0603 -> Resistor:RESISTOR0805
- R3: value R3 -> 10k; device resistor:R-US_R0603 -> Resistor:RESISTOR0805
- R4, R8: value 10k -> 100; device adafruit:R-US_R0603 -> Resistor:RESISTOR0805
- R5, R6: value 1k -> 10k; device resistor:R-US_R0603 -> Resistor:RESISTOR0805
- R7: device resistor:R-US_R0603 -> Resistor:RESISTOR0805
- R9: device adafruit:R-US_R0603 -> Resistor:RESISTOR0805
Connections:
- removed net ESTOP: IC1A.I1, IC1B.I1, IC1C.I1, JP2.5, R4.2
- removed net IN1: IC1A.I0, JP2.2, R10.2
- removed net IN2: IC1B.I0, JP2.3, R9.2
- removed net IN3: IC1C.I0, JP2.4, R8.2
- removed net OUT1: D1.C, F1.1, U1.D
- removed net OUT2: D2.C, F2.1, U2.D
- removed net OUT3: D3.C, F3.1, U3.D
- removed net VDD: C1.1, JP2.1
- removed net VSS: C1.2, JP2.6, R10.1, R4.1, R8.1, R9.1
- new net 1_H: J1.1, U$1.1
- new net 1_L: ETH2.1, Q1.D
- new net 2_H: J1.3, U$2.1
- new net 2_L: ETH2.3, Q2.D
- new net 3_H: J1.5, U$3.1
- new net 3_L: ETH2.5, Q3.D
- new net 4_H: J2.1, U$4.1
- new net 4_L: ETH2.7, Q4.D
- new net 5_H: J2.3, U$5.1
- new net 5_L: ETH1.1, Q5.D
- new net 6_H: J2.5, U$6.1
- new net 6_L: ETH1.3, Q6.D
- new net 7_H: J3.1, U$7.1
- new net 7_L: ETH1.5, Q7.D
- new net AUX_12V: E1.3, E1.4, J1.4, J2.2, J2.6, J3.4
- new net AUX_5V: E1.2, E1.5, J3.3
- new net FC_12V: E2.3, E2.4, J1.2, J1.6, J2.4, J3.2, J3.6
- new net FC_5V: E2.2, E2.5, J3.5, R3.1, R6.1, U$10.VCC, U$11.VCC, U$12.VCC, U$13.VCC, U$14.VCC, U$15.VCC, U$16.VCC, U$17.VCC, U$18.VCC, U$19.VCC, U$20.VCC, U$21.VCC, U$8.VCC, U$9.VCC
- new net GND_ISOLATED: ETH3.8, U$10.CAT, U$12.CAT, U$14.CAT, U$16.CAT, U$18.CAT, U$20.CAT, U$8.CAT
- new net IN_1: ETH3.1, R7.2
- new net IN_2: ETH3.2, R10.2
- new net IN_3: ETH3.3, R17.2
- new net IN_4: ETH3.4, R16.2
- new net IN_5: ETH3.5, R15.2
- new net IN_6: ETH3.6, R22.2
- new net IN_7: ETH3.7, R23.2
- new net N$13: Q3.G, R8.2, R9.2
- new net N$14: Q4.G, R11.2, R12.2
- new net N$15: Q5.G, R14.2
- new net N$16: Q6.G, R18.2, R19.2
- new net N$17: R6.2, U$10.VOUT, U$11.IN
- new net N$18: R4.2, U$11.OUT
- new net N$19: Q7.G, R20.2, R21.2
- new net N$20: R17.1, U$12.AN
- new net N$21: R16.1, U$14.AN
- new net N$22: R15.1, U$16.AN
- new net N$23: R22.1, U$18.AN
- new net N$24: R23.1, U$20.AN
- new net N$25: R10.1, U$10.AN
- new net N$26: R7.1, U$8.AN
- new net N$29: U$12.VOUT, U$13.IN
- new net N$3: ETH2.4, U$2.2
- new net N$30: R8.1, U$13.OUT
- new net N$38: U$16.VOUT, U$17.IN
- new net N$41: R14.1, U$17.OUT
- new net N$46: U$14.VOUT, U$15.IN
- new net N$47: R12.1, U$15.OUT
- new net N$5: ETH2.8, U$4.2
- new net N$54: U$20.VOUT, U$21.IN
- new net N$59: R21.1, U$21.OUT
- new net N$64: U$18.VOUT, U$19.IN
- new net N$67: R19.1, U$19.OUT
- net GND: now also E1.1, E1.6, E1.SH1, E1.SH2, E2.1, E2.6, E2.SH1, E2.SH2, ETH1.SHD1, ETH1.SHD2, ETH2.SHD1, ETH2.SHD2, ETH3.SHD1, ETH3.SHD2, Q1.S, Q2.S, Q3.S, Q4.S, Q5.S, Q6.S, Q7.S, R11.1, R13.1, R18.1, R2.2, R20.1, R5.2, R9.1, U$10.GND, U$11.GND, U$12.GND, U$13.GND, U$14.GND, U$15.GND, U$16.GND, U$17.GND, U$18.GND, U$19.GND, U$20.GND, U$21.GND, U$8.GND, U$9.GND; no longer D1.A, D2.A, D3.A, JP1.2, JP1.4, JP1.6, R1.1, R2.1, R3.1, R5.1, R6.1, R7.1, U1.S, U2.S, U3.S
- net N$1: now also ETH2.2, U$1.2; no longer IC1A.O, LED1.A, R1.2, U1.G
- net N$10: now also ETH1.6, U$7.2; no longer LED1.C, R5.2
- net N$11: now also ETH1.4, U$6.2; no longer LED2.C, R6.2
- net N$12: now also Q2.G, R4.1, R5.1; no longer LED3.C, R7.2
- net N$4: now also ETH2.6, U$3.2; no longer IC1B.O, LED2.A, R2.2, U2.G
- net N$6: now also ETH1.2, U$5.2; no longer IC1C.O, LED3.A, R3.2, U3.G
- net N$7: now also Q1.G, R1.1, R2.1; no longer F1.2, JP1.1
- net N$8: now also R3.2, U$8.VOUT, U$9.IN; no longer F2.2, JP1.3
- net N$9: now also R1.2, U$9.OUT; no longer F3.2, JP1.5
Other:
- note added: "Reegan McAllister"
